Commit message: fixed robotics function abstraction

File: urdf/rb10_1300e_DDA.urdf (robot description, URDF)
Before this commit: robot dda_rb10_1300e, 11 links, 10 joints
Links:
- removed link dda_link_tcp
- link dda_link_carriage: geometry collision box size=0.4 0.5 1.0; visual box size=0.4 0.7 1.0
Joints:
- removed joint dda_joint_tcp
- joint dda_joint_carriage: limit lower=0.0 upper=0.5 effort=1000.0 velocity=1.0 -> lower=-1 upper=1 effort=1000.0 velocity=1.0; origin xyz=0.2 0 0.2 rpy=0 0 0 -> xyz=0.2 0 0.5 rpy=0 0 0
- joint dda_joint_linear_track: origin xyz=0 0 0.2 rpy=0 0 0 -> xyz=0 0 0.7 rpy=0 0 0

File: urdf/rb20_1900es_RT.urdf (robot description, URDF)
Before this commit: robot rt_rb20_1900es, 11 links, 10 joints
Links:
- removed link rt_tcp
Joints:
- removed joint rt_tcp_joint
- joint rt_joint_carriage: limit lower=0.0 upper=0.5 effort=1000.0 velocity=1.0 -> lower=-1 upper=1 effort=1000.0 velocity=1.0
